File: pcb_stator-project/pcb_stator-project.kicad_pcb (KiCad board)
At the start: 2 copper layers, 4 parts, among them J1 PH_A, J2 PH_B, J3 PH_0, J4 PH_C

Commit message: wip
Parts:
- moved J1 149.8 mm to (254.2, 76.7)
- moved J4 149.8 mm to (262.2, 64.7)
- moved J2 149.8 mm to (268.6, 64.7)
- moved J3 149.8 mm to (263.0, 86.0)
Routing:
- net (no net): track 0.00 -> 1332.0 mm, vias 0 -> 12
Changed lines of the file:
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@@
   (setup
     (pad_to_mask_clearance 0)
+    (aux_axis_origin 100 100)
     (pcbplotparams
       (layerselection 0x00010fc_ffffffff)
@@
   (net 1 "Net-(J1-Pad1)")
   (footprint "Connector_Wire:SolderWire-2sqmm_1x01_D2mm_OD3.9mm" (layer "F.Cu")
-    (at 112.3712 63.2904)
+    (at 262.1888 64.7338)
     (descr "Soldered wire connection, for a single 2 mm² wire, reinforced insulation, conductor diameter 2mm, outer diameter 3.9mm, size source Multi-Contact FLEXI-xV 2.0 (https://ec.staubli.com/AcroFiles/Catalogues/TM_Cab-Main-11014119_(en)_hi.pdf), bend radius 3 times outer diameter, generated with kicad-footprint-generator")
     (tags "connector wire 2sqmm")
@@
   )
   (footprint "Connector_Wire:SolderWire-2sqmm_1x01_D2mm_OD3.9mm" (layer "F.Cu")
-    (at 113.1824 84.5566)
+    (at 263 86)
     (descr "Soldered wire connection, for a single 2 mm² wire, reinforced insulation, conductor diameter 2mm, outer diameter 3.9mm, size source Multi-Contact FLEXI-xV 2.0 (https://ec.staubli.com/AcroFiles/Catalogues/TM_Cab-Main-11014119_(en)_hi.pdf), bend radius 3 times outer diameter, generated with kicad-footprint-generator")
     (tags "connector wire 2sqmm")
@@
   )
   (footprint "Connector_Wire:SolderWire-2sqmm_1x01_D2mm_OD3.9mm" (layer "F.Cu")
-    (at 104.3686 75.2094)
+    (at 254.1862 76.6528)
     (descr "Soldered wire connection, for a single 2 mm² wire, reinforced insulation, conductor diameter 2mm, outer diameter 3.9mm, size source Multi-Contact FLEXI-xV 2.0 (https://ec.staubli.com/AcroFiles/Catalogues/TM_Cab-Main-11014119_(en)_hi.pdf), bend radius 3 times outer diameter, generated with kicad-footprint-generator")
     (tags "connector wire 2sqmm")
@@
   )
   (footprint "Connector_Wire:SolderWire-2sqmm_1x01_D2mm_OD3.9mm" (layer "F.Cu")
-    (at 118.8212 63.2904)
+    (at 268.6388 64.7338)
     (descr "Soldered wire connection, for a single 2 mm² wire, reinforced insulation, conductor diameter 2mm, outer diameter 3.9mm, size source Multi-Contact FLEXI-xV 2.0 (https://ec.staubli.com/AcroFiles/Catalogues/TM_Cab-Main-11014119_(en)_hi.pdf), bend radius 3 times outer diameter, generated with kicad-footprint-generator")
     (tags "connector wire 2sqmm")
@@
     )
   )
+  (segment (start 21.928203 21.980762) (end 22.928203 23.712812) (width 1) (layer "F.Cu") (net 0))
+  (segment (start -30 -9.999999) (end -30 8) (width 1) (layer "F.Cu") (net 0))
+  (segment (start 30 -8) (end 32 -8) (width 1) (layer "F.Cu") (net 0))
+  (segment (start -26.339745 65.621778) (end -43.660254 55.621778) (width 1) (layer "F.Cu") (net 0))
+  (segment (start -22.928203 23.712812) (end -10.803847 30.712812) (width 1) (layer "F.Cu") (net 0))
+  (segment (start -22.928203 -23.712812) (end -40.928203 -54.889727) (width 1) (layer "F.Cu") (net 0))
+  (segment (start -6.339745 -30.980762) (end -21.928203 -21.980762) (width 1) (layer "F.Cu") (net 0))
+  (segment (start 23.660254 20.980762) (end 43.660254 55.621778) (width 1) (layer "F.Cu") (net 0))
+  (segment (start 70 10) (end 30 10) (width 1) (layer "F.Cu") (net 0))
+  (segment (start 6.339745 -30.980762) (end 26.339745 -65.621778) (width 1) (layer "F.Cu") (net 0))
+  (segment (start -70 -9.999999) (end -30 -9.999999) (width 1) (layer "F.Cu") (net 0))
+  (segment (start -27.071796 -62.889727) (end -9.071796 -31.712812) (width 1) (layer "F.Cu") (net 0))
+  (segment (start 9.071796 31.712812) (end 21.196152 24.712812) (width 1) (layer "F.Cu") (net 0))
+  (segment (start -68 -7.999999) (end -32 -7.999999) (width 1) (layer "F.Cu") (net 0))
+  (segment (start -40.928203 54.889727) (end -22.928203 23.712812) (width 1) (layer "F.Cu") (net 0))
+  (segment (start -23.660254 -20.980762) (end -43.660254 -55.621778) (width 1) (layer "F.Cu") (net 0))
+  (segment (start -26.339745 -65.621778) (end -6.339745 -30.980762) (width 1) (layer "F.Cu") (net 0))
+  (segment (start 43.660254 -55.621778) (end 23.660254 -20.980762) (width 1) (layer "F.Cu") (net 0))
+  (segment (start 30 -10) (end 70 -10) (width 1) (layer "F.Cu") (net 0))
+  (segment (start 8.071796 -29.980762) (end 9.071796 -31.712812) (width 1) (layer "F.Cu") (net 0))
+  (segment (start 30 10) (end 30 -8) (width 1) (layer "F.Cu") (net 0))
+  (segment (start -32 -7.999999) (end -32 6) (width 1) (layer "F.Cu") (net 0))
+  (segment (start -68 8) (end -68 -7.999999) (width 1) (layer "F.Cu") (net 0))
+  (segment (start 22.928203 -23.712812) (end 10.803847 -30.712812) (width 1) (layer "F.Cu") (net 0))
+  (segment (start -27.071796 62.889727) (end -40.928203 54.889727) (width 1) (layer "F.Cu") (net 0))
+  (segment (start 9.071796 -31.712812) (end 27.071796 -62.889727) (width 1) (layer "F.Cu") (net 0))
+  (segment (start -43.660254 -55.621778) (end -26.339745 -65.621778) (width 1) (layer "F.Cu") (net 0))
+  (segment (start 68 8) (end 32 8) (width 1) (layer "F.Cu") (net 0))
+  (segment (start -9.071796 -31.712812) (end -21.196152 -24.712812) (width 1) (layer "F.Cu") (net 0))
+  (segment (start -8.071796 29.980762) (end -9.071796 31.712812) (width 1) (layer "F.Cu") (net 0))
+  (segment (start 40.928203 -54.889727) (end 22.928203 -23.712812) (width 1) (layer "F.Cu") (net 0))
+  (segment (start -21.928203 -21.980762) (end -22.928203 -23.712812) (width 1) (layer "F.Cu") (net 0))
+  (segment (start 32 8) (end 32 -6) (width 1) (layer "F.Cu") (net 0))
+  (segment (start 40.928203 54.889727) (end 27.071796 62.889727) (width 1) (layer "F.Cu") (net 0))
+  (segment (start 27.071796 62.889727) (end 9.071796 31.712812) (width 1) (layer "F.Cu") (net 0))
+  (segment (start 23.660254 -20.980762) (end 8.071796 -29.980762) (width 1) (layer "F.Cu") (net 0))
+  (segment (start 27.071796 -62.889727) (end 40.928203 -54.889727) (width 1) (layer "F.Cu") (net 0))
+  (segment (start -9.071796 31.712812) (end -27.071796 62.889727) (width 1) (layer "F.Cu") (net 0))
+  (segment (start -23.660254 20.980762) (end -8.071796 29.980762) (width 1) (layer "F.Cu") (net 0))
+  (segment (start 6.339745 30.980762) (end 21.928203 21.980762) (width 1) (layer "F.Cu") (net 0))
+  (segment (start -40.928203 -54.889727) (end -27.071796 -62.889727) (width 1) (layer "F.Cu") (net 0))
+  (segment (start -6.339745 30.980762) (end -26.339745 65.621778) (width 1) (layer "F.Cu") (net 0))
+  (segment (start 68 -8) (end 68 8) (width 1) (layer "F.Cu") (net 0))
+  (segment (start 43.660254 55.621778) (end 26.339745 65.621778) (width 1) (layer "F.Cu") (net 0))
+  (segment (start 26.339745 -65.621778) (end 43.660254 -55.621778) (width 1) (layer "F.Cu") (net 0))
+  (segment (start -30 8) (end -32 8) (width 1) (layer "F.Cu") (net 0))
+  (segment (start -30 10) (end -70 10) (width 1) (layer "F.Cu") (net 0))
+  (segment (start 32 -8) (end 68 -8) (width 1) (layer "F.Cu") (net 0))
+  (segment (start -43.660254 55.621778) (end -23.660254 20.980762) (width 1) (layer "F.Cu") (net 0))
+  (segment (start 22.928203 23.712812) (end 40.928203 54.889727) (width 1) (layer "F.Cu") (net 0))
+  (segment (start -70 10) (end -70 -9.999999) (width 1) (layer "F.Cu") (net 0))
+  (segment (start 26.339745 65.621778) (end 6.339745 30.980762) (width 1) (layer "F.Cu") (net 0))
+  (segment (start 70 -10) (end 70 10) (width 1) (layer "F.Cu") (net 0))
+  (segment (start -32 8) (end -68 8) (width 1) (layer "F.Cu") (net 0))
+  (via (at -21.196152 -24.712812) (size 2) (drill 1) (layers "F.Cu" "B.Cu") (net 0))
+  (via (at -30 10) (size 2) (drill 1) (layers "F.Cu" "B.Cu") (net 0))
+  (via (at 6.339745 -30.980762) (size 2) (drill 1) (layers "F.Cu" "B.Cu") (net 0))
+  (via (at 21.196152 24.712812) (size 2) (drill 1) (layers "F.Cu" "B.Cu") (net 0))
+  (via (at 10.803847 -30.712812) (size 2) (drill 1) (layers "F.Cu" "B.Cu") (net 0))
+  (via (at 30 -10) (size 2) (drill 1) (layers "F.Cu" "B.Cu") (net 0))
+  (via (at -32 6) (size 2) (drill 1) (layers "F.Cu" "B.Cu") (net 0))
+  (via (at -10.803847 30.712812) (size 2) (drill 1) (layers "F.Cu" "B.Cu") (net 0))
+  (via (at -6.339745 30.980762) (size 2) (drill 1) (layers "F.Cu" "B.Cu") (net 0))
+  (via (at 23.660254 20.980762) (size 2) (drill 1) (layers "F.Cu" "B.Cu") (net 0))
+  (via (at -23.660254 -20.980762) (size 2) (drill 1) (layers "F.Cu" "B.Cu") (net 0))
+  (via (at 32 -6) (size 2) (drill 1) (layers "F.Cu" "B.Cu") (net 0))
 )

Commit message: gui working
Routing:
- net (no net): track 1332.0 -> 0.00 mm, vias 12 -> 0
Changed lines of the file:
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@@
     )
   )
-  (segment (start 21.928203 21.980762) (end 22.928203 23.712812) (width 1) (layer "F.Cu") (net 0))
-  (segment (start -30 -9.999999) (end -30 8) (width 1) (layer "F.Cu") (net 0))
-  (segment (start 30 -8) (end 32 -8) (width 1) (layer "F.Cu") (net 0))
-  (segment (start -26.339745 65.621778) (end -43.660254 55.621778) (width 1) (layer "F.Cu") (net 0))
-  (segment (start -22.928203 23.712812) (end -10.803847 30.712812) (width 1) (layer "F.Cu") (net 0))
-  (segment (start -22.928203 -23.712812) (end -40.928203 -54.889727) (width 1) (layer "F.Cu") (net 0))
-  (segment (start -6.339745 -30.980762) (end -21.928203 -21.980762) (width 1) (layer "F.Cu") (net 0))
-  (segment (start 23.660254 20.980762) (end 43.660254 55.621778) (width 1) (layer "F.Cu") (net 0))
-  (segment (start 70 10) (end 30 10) (width 1) (layer "F.Cu") (net 0))
-  (segment (start 6.339745 -30.980762) (end 26.339745 -65.621778) (width 1) (layer "F.Cu") (net 0))
-  (segment (start -70 -9.999999) (end -30 -9.999999) (width 1) (layer "F.Cu") (net 0))
-  (segment (start -27.071796 -62.889727) (end -9.071796 -31.712812) (width 1) (layer "F.Cu") (net 0))
-  (segment (start 9.071796 31.712812) (end 21.196152 24.712812) (width 1) (layer "F.Cu") (net 0))
-  (segment (start -68 -7.999999) (end -32 -7.999999) (width 1) (layer "F.Cu") (net 0))
-  (segment (start -40.928203 54.889727) (end -22.928203 23.712812) (width 1) (layer "F.Cu") (net 0))
-  (segment (start -23.660254 -20.980762) (end -43.660254 -55.621778) (width 1) (layer "F.Cu") (net 0))
-  (segment (start -26.339745 -65.621778) (end -6.339745 -30.980762) (width 1) (layer "F.Cu") (net 0))
-  (segment (start 43.660254 -55.621778) (end 23.660254 -20.980762) (width 1) (layer "F.Cu") (net 0))
-  (segment (start 30 -10) (end 70 -10) (width 1) (layer "F.Cu") (net 0))
-  (segment (start 8.071796 -29.980762) (end 9.071796 -31.712812) (width 1) (layer "F.Cu") (net 0))
-  (segment (start 30 10) (end 30 -8) (width 1) (layer "F.Cu") (net 0))
-  (segment (start -32 -7.999999) (end -32 6) (width 1) (layer "F.Cu") (net 0))
-  (segment (start -68 8) (end -68 -7.999999) (width 1) (layer "F.Cu") (net 0))
-  (segment (start 22.928203 -23.712812) (end 10.803847 -30.712812) (width 1) (layer "F.Cu") (net 0))
-  (segment (start -27.071796 62.889727) (end -40.928203 54.889727) (width 1) (layer "F.Cu") (net 0))
-  (segment (start 9.071796 -31.712812) (end 27.071796 -62.889727) (width 1) (layer "F.Cu") (net 0))
-  (segment (start -43.660254 -55.621778) (end -26.339745 -65.621778) (width 1) (layer "F.Cu") (net 0))
-  (segment (start 68 8) (end 32 8) (width 1) (layer "F.Cu") (net 0))
-  (segment (start -9.071796 -31.712812) (end -21.196152 -24.712812) (width 1) (layer "F.Cu") (net 0))
-  (segment (start -8.071796 29.980762) (end -9.071796 31.712812) (width 1) (layer "F.Cu") (net 0))
-  (segment (start 40.928203 -54.889727) (end 22.928203 -23.712812) (width 1) (layer "F.Cu") (net 0))
-  (segment (start -21.928203 -21.980762) (end -22.928203 -23.712812) (width 1) (layer "F.Cu") (net 0))
-  (segment (start 32 8) (end 32 -6) (width 1) (layer "F.Cu") (net 0))
-  (segment (start 40.928203 54.889727) (end 27.071796 62.889727) (width 1) (layer "F.Cu") (net 0))
-  (segment (start 27.071796 62.889727) (end 9.071796 31.712812) (width 1) (layer "F.Cu") (net 0))
-  (segment (start 23.660254 -20.980762) (end 8.071796 -29.980762) (width 1) (layer "F.Cu") (net 0))
-  (segment (start 27.071796 -62.889727) (end 40.928203 -54.889727) (width 1) (layer "F.Cu") (net 0))
-  (segment (start -9.071796 31.712812) (end -27.071796 62.889727) (width 1) (layer "F.Cu") (net 0))
-  (segment (start -23.660254 20.980762) (end -8.071796 29.980762) (width 1) (layer "F.Cu") (net 0))
-  (segment (start 6.339745 30.980762) (end 21.928203 21.980762) (width 1) (layer "F.Cu") (net 0))
-  (segment (start -40.928203 -54.889727) (end -27.071796 -62.889727) (width 1) (layer "F.Cu") (net 0))
-  (segment (start -6.339745 30.980762) (end -26.339745 65.621778) (width 1) (layer "F.Cu") (net 0))
-  (segment (start 68 -8) (end 68 8) (width 1) (layer "F.Cu") (net 0))
-  (segment (start 43.660254 55.621778) (end 26.339745 65.621778) (width 1) (layer "F.Cu") (net 0))
-  (segment (start 26.339745 -65.621778) (end 43.660254 -55.621778) (width 1) (layer "F.Cu") (net 0))
-  (segment (start -30 8) (end -32 8) (width 1) (layer "F.Cu") (net 0))
-  (segment (start -30 10) (end -70 10) (width 1) (layer "F.Cu") (net 0))
-  (segment (start 32 -8) (end 68 -8) (width 1) (layer "F.Cu") (net 0))
-  (segment (start -43.660254 55.621778) (end -23.660254 20.980762) (width 1) (layer "F.Cu") (net 0))
-  (segment (start 22.928203 23.712812) (end 40.928203 54.889727) (width 1) (layer "F.Cu") (net 0))
-  (segment (start -70 10) (end -70 -9.999999) (width 1) (layer "F.Cu") (net 0))
-  (segment (start 26.339745 65.621778) (end 6.339745 30.980762) (width 1) (layer "F.Cu") (net 0))
-  (segment (start 70 -10) (end 70 10) (width 1) (layer "F.Cu") (net 0))
-  (segment (start -32 8) (end -68 8) (width 1) (layer "F.Cu") (net 0))
-  (via (at -21.196152 -24.712812) (size 2) (drill 1) (layers "F.Cu" "B.Cu") (net 0))
-  (via (at -30 10) (size 2) (drill 1) (layers "F.Cu" "B.Cu") (net 0))
-  (via (at 6.339745 -30.980762) (size 2) (drill 1) (layers "F.Cu" "B.Cu") (net 0))
-  (via (at 21.196152 24.712812) (size 2) (drill 1) (layers "F.Cu" "B.Cu") (net 0))
-  (via (at 10.803847 -30.712812) (size 2) (drill 1) (layers "F.Cu" "B.Cu") (net 0))
-  (via (at 30 -10) (size 2) (drill 1) (layers "F.Cu" "B.Cu") (net 0))
-  (via (at -32 6) (size 2) (drill 1) (layers "F.Cu" "B.Cu") (net 0))
-  (via (at -10.803847 30.712812) (size 2) (drill 1) (layers "F.Cu" "B.Cu") (net 0))
-  (via (at -6.339745 30.980762) (size 2) (drill 1) (layers "F.Cu" "B.Cu") (net 0))
-  (via (at 23.660254 20.980762) (size 2) (drill 1) (layers "F.Cu" "B.Cu") (net 0))
-  (via (at -23.660254 -20.980762) (size 2) (drill 1) (layers "F.Cu" "B.Cu") (net 0))
-  (via (at 32 -6) (size 2) (drill 1) (layers "F.Cu" "B.Cu") (net 0))
 )

Commit message: terminals POC ok
Parts:
- moved J4 272.4 mm to (-2.00, 131.0)
- moved J2 270.9 mm to (6.00, 131.0)
- moved J3 270.4 mm to (-2.00, 140.0)
- moved J1 269.7 mm to (-10.0, 131.0)
Routing:
- net (no net): track 0.00 -> 20999.1 mm, vias 0 -> 27
