File: kimotor-project/kimotor-6-jlcpcb.kicad_pcb (KiCad board)
At the start: 6 copper layers, 0 parts

Commit message: 6 layers connections draft OK
Parts:
- added ?: MountingHole_3.2mm_M3_Pad, MountingHole_3.2mm_M3_Pad, F.Cu at (-23.7, 41.1)
- added ?: Pin_D1.0mm_L10.0mm, Pin_D1.0mm_L10.0mm, F.Cu at (3.75, 42.8)
- added ?: Pin_D1.0mm_L10.0mm, Pin_D1.0mm_L10.0mm, F.Cu at (0.00, 43.0)
- added ?: Pin_D1.0mm_L10.0mm, Pin_D1.0mm_L10.0mm, F.Cu at (-3.75, 42.8)
- added ?: MountingHole_3.2mm_M3_Pad, MountingHole_3.2mm_M3_Pad, F.Cu at (23.7, -41.1)
- added ?: MountingHole_3.2mm_M3_Pad, MountingHole_3.2mm_M3_Pad, F.Cu at (-23.8, -41.1)
- added ?: MountingHole_3.2mm_M3_Pad, MountingHole_3.2mm_M3_Pad, F.Cu at (-47.5, 0.00)
- added ?: MountingHole_3.2mm_M3_Pad, MountingHole_3.2mm_M3_Pad, F.Cu at (47.5, 0.00)
- added ?: MountingHole_3.2mm_M3_Pad, MountingHole_3.2mm_M3_Pad, F.Cu at (23.8, 41.1)
Routing:
- net (no net): track 0.00 -> 99987.3 mm, vias 0 -> 36
- net gnd: vias 0 -> 96
- added copper zone on B.Cu, net gnd
- added copper zone on F.Cu, net gnd
- added copper zone on In1.Cu, net gnd
- added copper zone on In2.Cu, net gnd
- added copper zone on In3.Cu, net gnd
- added copper zone on In4.Cu, net gnd
