File: kimotor-project/kimotor-project.kicad_pcb (KiCad board)
At the start: 4 copper layers, 0 parts

Commit message: WIP junctions
Routing:
- net (no net): track 26014.8 -> 0.00 mm, vias 6 -> 0

Commit message: working holes
Routing:
- net (no net): track 0.00 -> 26014.8 mm, vias 0 -> 6
