File: kimotor-project/kimotor-project.kicad_pcb (KiCad board)
At the start: 4 copper layers, 0 parts

Commit message: improved thermals, silk WIP
Parts:
- added ?: Pin_D1.0mm_L10.0mm, Pin_D1.0mm_L10.0mm, F.Cu at (-3.79, 43.3)
- added ?: MountingHole_3.2mm_M3_Pad, MountingHole_3.2mm_M3_Pad, F.Cu at (-23.8, -41.1)
- added ?: Pin_D1.0mm_L10.0mm, Pin_D1.0mm_L10.0mm, F.Cu at (3.79, 43.3)
- added ?: MountingHole_3.2mm_M3_Pad, MountingHole_3.2mm_M3_Pad, F.Cu at (-47.5, 0.00)
- added ?: MountingHole_3.2mm_M3_Pad, MountingHole_3.2mm_M3_Pad, F.Cu at (23.7, -41.1)
- added ?: MountingHole_3.2mm_M3_Pad, MountingHole_3.2mm_M3_Pad, F.Cu at (-23.7, 41.1)
- added ?: Pin_D1.0mm_L10.0mm, Pin_D1.0mm_L10.0mm, F.Cu at (0.00, 43.5)
- added ?: MountingHole_3.2mm_M3_Pad, MountingHole_3.2mm_M3_Pad, F.Cu at (23.8, 41.1)
- added ?: MountingHole_3.2mm_M3_Pad, MountingHole_3.2mm_M3_Pad, F.Cu at (47.5, 0.00)
Routing:
- net (no net): track 0.00 -> 7802.9 mm, vias 0 -> 12
- net gnd: vias 0 -> 72
- added copper zone on B.Cu, net gnd
- added copper zone on F.Cu, net gnd
