File: kimotor-project/kimotor-project.kicad_pcb (KiCad board)
At the start: 4 copper layers, 9 parts

Commit message: jlcpcb test run
Routing:
- net (no net): track 7802.9 -> 8100.5 mm
Other:
- copper layers 4 -> 2

Commit message: polished resources
Parts:
- removed ? (x6): MountingHole_3.2mm_M3_Pad, MountingHole_3.2mm_M3_Pad
- removed ? (x3): Pin_D1.0mm_L10.0mm, Pin_D1.0mm_L10.0mm
Routing:
- net (no net): track 8100.5 -> 0.00 mm, vias 12 -> 0
- net gnd: vias 72 -> 0
- removed copper zone on B.Cu, net gnd
- removed copper zone on F.Cu, net gnd
Other:
- copper layers 2 -> 6

Commit message: kimotor_pro: bump to v8 + use some JLCPCB capabilities
Other:
- copper layers 6 -> 8
- board text added: "20240429_ly8_s6_w10"
